File: Expansion_01.brd (EAGLE design)
At the start: 100 x 80 mm, 26 parts, among them U1 W65C22_01, U2 W65C22_02, X1 2550-

Commit message: Finished schematics
Finished schematics
Parts:
- added C1, C2: 10uF, rcl:E2-5
- added IC1: LD1086-33, linear:TO220H
- added IC2: P8X32A-D40DIP-40, propeller-dip-plus:P8X32A-D40
- added IC3: 24LC256DIP-8, propeller-dip-plus:24LC256
- added JP1: Programming port, pinhead:1X04/90
- added LED2: 5MM-LED, propeller-dip-plus:5MM-LED
- added LINE: Line Out, con-lumberg:1503_04
- added R10: 330, resistor:0207/10
- added R12, R13: 10K, resistor:0207/10
- added R14, R15, R16, R17, R18, R19, R20, R21, R22, R23, R24, R25, R26, R27, R28, R29: 1K, resistor:0207/10
- added R30, R31, R32, R34, R36: 240, resistor:0207/10
- added R33, R35, R37: 470, resistor:0207/10
- added VGA: VGA Connector, HD15_B:HD15F
- added XTAL1: 5MHZ, propeller-dip-plus:5MHZ-CRYSTAL
- D10, D9: value 1N4148 -> 1N5817; device diode:DO35-7 -> diode:DO41-7.6
- moved D9 161.9 mm to (3.81, -120.7), turned to 0 degrees
- moved D10 160.2 mm to (3.81, -128.3), turned to 0 degrees
Connections:
- new net +3V3: C2.+, IC1.2, IC2.12, IC2.32, IC3.8, R10.1, R12.2, R13.2
- new net N$25: LED2.A, R10.2
- new net N$26: IC2.40, JP1.3
- new net N$27: IC2.39, JP1.4
- new net N$28: IC2.31, XTAL1.2
- new net N$29: IC2.30, XTAL1.1
- new net N$30: IC2.11, JP1.2
- new net N$31: IC2.38, IC3.5, R13.1
- new net N$32: IC2.37, IC3.6, R12.1
- new net N$33: IC2.1, R14.2
- new net N$34: IC2.2, R15.2
- new net N$35: IC2.3, R16.2
- new net N$36: IC2.4, R17.2
- new net N$37: IC2.5, R18.2
- new net N$38: IC2.6, R19.2
- new net N$39: IC2.7, R20.2
- new net N$40: IC2.8, R21.2
- new net N$41: IC2.13, R22.2
- new net N$42: IC2.14, R23.2
- new net N$43: IC2.15, R24.2
- new net N$44: IC2.16, R25.2
- new net N$45: IC2.17, R26.2
- new net N$46: IC2.18, R27.2
- new net N$47: IC2.19, R28.2
- new net N$48: IC2.20, R29.2
- new net N$49: R32.1, R33.1, VGA.1
- new net N$50: R34.1, R35.1, VGA.2
- new net N$51: R36.1, R37.1, VGA.3
- new net N$52: IC2.23, R37.2
- new net N$53: IC2.22, R31.1
- new net N$54: R30.2, VGA.14
- new net N$55: R31.2, VGA.13
- new net N$56: IC2.21, R30.1
- new net N$57: IC2.24, R36.2
- new net N$58: IC2.25, R35.2
- new net N$59: IC2.26, R34.2
- new net N$60: IC2.27, R33.2
- new net N$61: IC2.28, R32.2
- new net N$62: IC2.33, LINE.1
- new net N$63: IC2.34, LINE.2
- new net U2_PA_0: R14.1, U2.2
- new net U2_PA_1: R15.1, U2.3
- new net U2_PA_2: R16.1, U2.4
- new net U2_PA_3: R17.1, U2.5
- new net U2_PA_4: R18.1, U2.6
- new net U2_PA_5: R19.1, U2.7
- new net U2_PA_6: R20.1, U2.8
- new net U2_PA_7: R21.1, U2.9
- new net U2_PB_0: R22.1, U2.10
- new net U2_PB_1: R23.1, U2.11
- new net U2_PB_2: R24.1, U2.12
- new net U2_PB_3: R25.1, U2.13
- new net U2_PB_4: R26.1, U2.14
- new net U2_PB_5: R27.1, U2.15
- new net U2_PB_6: R28.1, U2.16
- new net U2_PB_7: R29.1, U2.17
- net N$20: now also D10.C; no longer D9.C
- net N$21: now also D9.C; no longer D10.C
- net VDD: now also C1.+, IC1.3
- net VSS: now also C1.-, C2.-, IC1.1, IC2.10, IC2.29, IC2.9, IC3.1, IC3.2, IC3.3, IC3.4, IC3.7, JP1.1, LED2.K, LINE.3, VGA.10, VGA.5, VGA.6, VGA.7, VGA.8, VGA.SH1, VGA.SH2
Routing:
- net VDD: track 153.7 -> 0.00 mm
- net U1_PA_1: track 83.1 -> 0.00 mm
- net N$1: track 81.7 -> 0.00 mm
- net U1_PA_0: track 75.0 -> 0.00 mm
- net RESB: track 72.4 -> 0.00 mm
- net U1_PA_2: track 70.6 -> 0.00 mm
- net U1_PA_4: track 67.3 -> 0.00 mm
- net U1_PA_3: track 64.3 -> 0.00 mm
- net PH2: track 64.0 -> 0.00 mm
- net VSS: track 61.5 -> 0.00 mm
- net DATA_BUS_7: track 56.4 -> 0.00 mm
- net U1_PA_5: track 55.6 -> 0.00 mm
- net DATA_BUS_5: track 54.3 -> 0.00 mm
- net U1_PA_6: track 50.8 -> 0.00 mm
- net ADDRESS_BUS_1: track 50.0 -> 0.00 mm, vias 1 -> 0
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
Commit message: Fixed Schematics
Fixed Schematics
Parts:
- added R38, R39: 10K, resistor:0207/10
Connections:
- net +3V3: now also R38.2, R39.2
- net N$26: now also R39.1
- net N$30: now also R38.1
Changed lines of the file:
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@@
 <attribute name="MF" value="" x="-8.89" y="-182.88" size="1.778" layer="27" display="off"/>
 </element>
+<element name="R38" library="resistor" package="0207/10" value="10K" x="-7.62" y="-199.39"/>
+<element name="R39" library="resistor" package="0207/10" value="10K" x="-7.62" y="-204.47"/>
 </elements>
 <signals>
@@
 <contactref element="R13" pad="2"/>
 <contactref element="R12" pad="2"/>
-<wire x1="26.67" y1="40.64" x2="41.91" y2="48.26" width="0" layer="19" extent="1-1"/>
-<wire x1="20.32" y1="39.37" x2="26.67" y2="40.64" width="0" layer="19" extent="1-1"/>
+<contactref element="R38" pad="2"/>
+<contactref element="R39" pad="2"/>
+<wire x1="-2.54" y1="-199.39" x2="-2.54" y2="-204.47" width="0" layer="19" extent="1-1"/>
+<wire x1="10.16" y1="-20.32" x2="-2.54" y2="-199.39" width="0" layer="19" extent="1-1"/>
+<wire x1="10.16" y1="-15.24" x2="10.16" y2="-20.32" width="0" layer="19" extent="1-1"/>
+<wire x1="17.78" y1="11.43" x2="10.16" y2="-15.24" width="0" layer="19" extent="1-1"/>
+<wire x1="20.32" y1="39.37" x2="17.78" y2="11.43" width="0" layer="19" extent="1-1"/>
+<wire x1="26.67" y1="40.64" x2="20.32" y2="39.37" width="0" layer="19" extent="1-1"/>
 <wire x1="20.066" y1="46.99" x2="20.32" y2="39.37" width="0" layer="19" extent="1-1"/>
 <wire x1="12.7" y1="52.07" x2="20.066" y2="46.99" width="0" layer="19" extent="1-1"/>
-<wire x1="17.78" y1="11.43" x2="20.32" y2="39.37" width="0" layer="19" extent="1-1"/>
-<wire x1="10.16" y1="-15.24" x2="17.78" y2="11.43" width="0" layer="19" extent="1-1"/>
-<wire x1="10.16" y1="-20.32" x2="10.16" y2="-15.24" width="0" layer="19" extent="1-1"/>
+<wire x1="41.91" y1="48.26" x2="26.67" y2="40.64" width="0" layer="19" extent="1-1"/>
 </signal>
 <signal name="N$25">
@@
 <contactref element="IC2" pad="11"/>
 <contactref element="JP1" pad="2"/>
-<wire x1="6.35" y1="-33.02" x2="26.67" y2="43.18" width="0" layer="19" extent="1-1"/>
+<contactref element="R38" pad="1"/>
+<wire x1="6.35" y1="-33.02" x2="-12.7" y2="-199.39" width="0" layer="19" extent="1-1"/>
+<wire x1="26.67" y1="43.18" x2="6.35" y2="-33.02" width="0" layer="19" extent="1-1"/>
 </signal>
 <signal name="N$31">
@@
 <contactref element="IC2" pad="40"/>
 <contactref element="JP1" pad="3"/>
-<wire x1="8.89" y1="-33.02" x2="41.91" y2="68.58" width="0" layer="19" extent="1-1"/>
+<contactref element="R39" pad="1"/>
+<wire x1="8.89" y1="-33.02" x2="-12.7" y2="-204.47" width="0" layer="19" extent="1-1"/>
+<wire x1="41.91" y1="68.58" x2="8.89" y2="-33.02" width="0" layer="19" extent="1-1"/>
 </signal>
 <signal name="N$27">
