File: Expansion_01.sch (EAGLE design)
At the start: 26 parts, among them U1 W65C22_01, U2 W65C22_02, X1 2550-

Commit message: Finished schematics
Finished schematics
Parts:
- added C1, C2: 10uF, rcl:CPOL-USE2-5
- added IC1: LD1086-33, linear:317T
- added IC2: P8X32A-D40DIP-40, propeller-dip-plus:P8X32A-D40DIP-40
- added IC3: 24LC256DIP-8, propeller-dip-plus:24LC256DIP-8
- added JP1: Programming port, pinhead:PINHD-1X4/90
- added LED2: 5MM-LED, propeller-dip-plus:5MM-LED
- added LINE: Line Out, con-lumberg:1503_04
- added R10: 330, resistor:R-US_0207/10
- added R12, R13: 10K, resistor:R-US_0207/10
- added R14, R15, R16, R17, R18, R19, R20, R21, R22, R23, R24, R25, R26, R27, R28, R29: 1K, resistor:R-US_0207/10
- added R30, R31, R32, R34, R36: 240, resistor:R-US_0207/10
- added R33, R35, R37: 470, resistor:R-US_0207/10
- added VGA: VGA Connector, HD15_B:VGAF
- added XTAL1: 5MHZ, propeller-dip-plus:5MHZ-CRYSTAL
- D10, D9: value 1N4148 -> 1N5817; device diode:1N4148DO35-7 -> diode:1N5817-B
Connections:
- new net +3V3: C2.+, IC1.VO, IC2.+3V3@1, IC2.+3V3@2, IC3.+3V3, R10.1, R12.2, R13.2
- new net N$25: LED2.A, R10.2
- new net N$26: IC2.P31, JP1.3
- new net N$27: IC2.P30, JP1.4
- new net N$28: IC2.XO, XTAL1.2
- new net N$29: IC2.XI, XTAL1.1
- new net N$30: IC2.RESN, JP1.2
- new net N$31: IC2.P29, IC3.SDA, R13.1
- new net N$32: IC2.P28, IC3.SCL, R12.1
- new net N$33: IC2.P0, R14.2
- new net N$34: IC2.P1, R15.2
- new net N$35: IC2.P2, R16.2
- new net N$36: IC2.P3, R17.2
- new net N$37: IC2.P4, R18.2
- new net N$38: IC2.P5, R19.2
- new net N$39: IC2.P6, R20.2
- new net N$40: IC2.P7, R21.2
- new net N$41: IC2.P8, R22.2
- new net N$42: IC2.P9, R23.2
- new net N$43: IC2.P10, R24.2
- new net N$44: IC2.P11, R25.2
- new net N$45: IC2.P12, R26.2
- new net N$46: IC2.P13, R27.2
- new net N$47: IC2.P14, R28.2
- new net N$48: IC2.P15, R29.2
- new net N$49: R32.1, R33.1, VGA.P$1
- new net N$50: R34.1, R35.1, VGA.P$2
- new net N$51: R36.1, R37.1, VGA.P$3
- new net N$52: IC2.P18, R37.2
- new net N$53: IC2.P17, R31.1
- new net N$54: R30.2, VGA.P$14
- new net N$55: R31.2, VGA.P$13
- new net N$56: IC2.P16, R30.1
- new net N$57: IC2.P19, R36.2
- new net N$58: IC2.P20, R35.2
- new net N$59: IC2.P21, R34.2
- new net N$60: IC2.P22, R33.2
- new net N$61: IC2.P23, R32.2
- new net N$62: IC2.P24, LINE.1
- new net N$63: IC2.P25, LINE.3
- new net U2_PA_0: R14.1, U2.PA0
- new net U2_PA_1: R15.1, U2.PA1
- new net U2_PA_2: R16.1, U2.PA2
- new net U2_PA_3: R17.1, U2.PA3
- new net U2_PA_4: R18.1, U2.PA4
- new net U2_PA_5: R19.1, U2.PA5
- new net U2_PA_6: R20.1, U2.PA6
- new net U2_PA_7: R21.1, U2.PA7
- new net U2_PB_0: R22.1, U2.PB0
- new net U2_PB_1: R23.1, U2.PB1
- new net U2_PB_2: R24.1, U2.PB2
- new net U2_PB_3: R25.1, U2.PB3
- new net U2_PB_4: R26.1, U2.PB4
- new net U2_PB_5: R27.1, U2.PB5
- new net U2_PB_6: R28.1, U2.PB6
- new net U2_PB_7: R29.1, U2.PB7
- net N$20: now also D10.C; no longer D9.C
- net N$21: now also D9.C; no longer D10.C
- net VDD: now also C1.+, IC1.VI
- net VSS: now also C1.-, C2.-, IC1.ADJ, IC2.BOEN, IC2.VSS@1, IC2.VSS@2, IC3.A0, IC3.A1, IC3.A2, IC3.VSS, IC3.WP, JP1.1, LED2.C, LINE.2, VGA.P$10, VGA.P$5, VGA.P$6, VGA.P$7, VGA.P$8, VGA.SH1, VGA.SH2

Commit message: Fixed Schematics
Fixed Schematics
Parts:
- added R38, R39: 10K, resistor:R-US_0207/10
Connections:
- net +3V3: now also R38.2, R39.2
- net N$26: now also R39.1
- net N$30: now also R38.1
Changed lines of the file:
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@@
 <setting verticaltext="up"/>
 </settings>
-<grid distance="0.05" unitdist="inch" unit="inch" style="lines" multiple="1" display="no" altdistance="0.01" altunitdist="inch" altunit="inch"/>
+<grid distance="0.1" unitdist="inch" unit="inch" style="lines" multiple="1" display="no" altdistance="0.01" altunitdist="inch" altunit="inch"/>
 <layers>
 <layer number="1" name="Top" color="4" fill="1" visible="no" active="no"/>
@@
 <part name="LINE" library="con-lumberg" deviceset="1503_04" device="" value="Line Out"/>
 <part name="VSS11" library="supply1" deviceset="VSS" device=""/>
+<part name="R38" library="resistor" deviceset="R-US_" device="0207/10" value="10K"/>
+<part name="+3V6" library="supply1" deviceset="+3V3" device=""/>
+<part name="R39" library="resistor" deviceset="R-US_" device="0207/10" value="10K"/>
 </parts>
 <sheets>
@@
 <instance part="IC3" gate="G$1" x="-17.78" y="194.31" rot="R270"/>
 <instance part="XTAL1" gate="G$1" x="16.51" y="147.32" rot="R90"/>
-<instance part="+3V5" gate="G$1" x="25.4" y="205.74"/>
+<instance part="+3V5" gate="G$1" x="25.4" y="215.9"/>
 <instance part="VSS7" gate="G$1" x="-33.02" y="185.42" smashed="yes">
 <attribute name="VALUE" x="-30.48" y="182.88" size="1.778" layer="96" rot="R180"/>
@@
 <attribute name="VALUE" x="72.39" y="50.8" size="1.778" layer="96" rot="R180"/>
 </instance>
+<instance part="R38" gate="G$1" x="-43.18" y="218.44" rot="R90"/>
+<instance part="+3V6" gate="G$1" x="-43.18" y="231.14"/>
+<instance part="R39" gate="G$1" x="17.78" y="205.74"/>
 </instances>
 <busses>
@@
 <pinref part="R12" gate="G$1" pin="2"/>
 <wire x1="25.4" y1="193.04" x2="25.4" y2="198.12" width="0.1524" layer="91"/>
-<wire x1="25.4" y1="198.12" x2="25.4" y2="203.2" width="0.1524" layer="91"/>
+<wire x1="25.4" y1="198.12" x2="25.4" y2="205.74" width="0.1524" layer="91"/>
+<wire x1="25.4" y1="205.74" x2="25.4" y2="213.36" width="0.1524" layer="91"/>
 <wire x1="22.86" y1="193.04" x2="25.4" y2="193.04" width="0.1524" layer="91"/>
 <junction x="25.4" y="193.04"/>
@@
 <wire x1="-7.62" y1="198.12" x2="25.4" y2="198.12" width="0.1524" layer="91"/>
 <junction x="25.4" y="198.12"/>
+<pinref part="R39" gate="G$1" pin="2"/>
+<wire x1="22.86" y1="205.74" x2="25.4" y2="205.74" width="0.1524" layer="91"/>
+<junction x="25.4" y="205.74"/>
 </segment>
 <segment>
@@
 <wire x1="12.7" y1="154.94" x2="12.7" y2="152.4" width="0.1524" layer="91"/>
 <wire x1="12.7" y1="152.4" x2="-5.08" y2="152.4" width="0.1524" layer="91"/>
+</segment>
+<segment>
+<pinref part="+3V6" gate="G$1" pin="+3V3"/>
+<pinref part="R38" gate="G$1" pin="2"/>
+<wire x1="-43.18" y1="228.6" x2="-43.18" y2="223.52" width="0.1524" layer="91"/>
 </segment>
 </net>
@@
 <wire x1="-50.8" y1="147.32" x2="-50.8" y2="210.82" width="0.1524" layer="91"/>
 <pinref part="JP1" gate="A" pin="2"/>
-<wire x1="-50.8" y1="210.82" x2="-15.24" y2="210.82" width="0.1524" layer="91"/>
+<wire x1="-50.8" y1="210.82" x2="-43.18" y2="210.82" width="0.1524" layer="91"/>
+<wire x1="-43.18" y1="210.82" x2="-15.24" y2="210.82" width="0.1524" layer="91"/>
 <wire x1="-15.24" y1="210.82" x2="-15.24" y2="223.52" width="0.1524" layer="91"/>
+<pinref part="R38" gate="G$1" pin="1"/>
+<wire x1="-43.18" y1="213.36" x2="-43.18" y2="210.82" width="0.1524" layer="91"/>
+<junction x="-43.18" y="210.82"/>
 </segment>
 </net>
@@
 <pinref part="IC2" gate="G$1" pin="P31"/>
 <wire x1="-5.08" y1="172.72" x2="2.54" y2="172.72" width="0.1524" layer="91"/>
-<wire x1="2.54" y1="172.72" x2="2.54" y2="210.82" width="0.1524" layer="91"/>
+<wire x1="2.54" y1="172.72" x2="2.54" y2="205.74" width="0.1524" layer="91"/>
 <pinref part="JP1" gate="A" pin="3"/>
+<wire x1="2.54" y1="205.74" x2="2.54" y2="210.82" width="0.1524" layer="91"/>
 <wire x1="2.54" y1="210.82" x2="-12.7" y2="210.82" width="0.1524" layer="91"/>
 <wire x1="-12.7" y1="210.82" x2="-12.7" y2="223.52" width="0.1524" layer="91"/>
-</segment>
-</net>
+<pinref part="R39" gate="G$1" pin="1"/>
+<wire x1="12.7" y1="205.74" x2="2.54" y2="205.74" width="0.1524" layer="91"/>
+<junction x="2.54" y="205.74"/>
+</segment>
+</net>
